Commit message: Add object contact labeling functionality and update URDF models
- Introduced inertial properties to the trashcan URDF model for better physics simulation.
- Added a new script to generate frame-level object-contact labels for HOI motion files, mapping intended contacts from SMPLH human joints to robot body names.
- Updated training command to include new contact labeling process and adjusted parameters for object contact thresholds and sampling ratios.
- Modified object parameters in YAML configuration to reflect updated mass distribution values.
- Created a new Python module for managing object contact utilities, including functions for resolving sample points and calculating distances to object surfaces.
- Added multiple labeled contact files for various objects, enhancing the dataset for training.

File: src/holosoma_retargeting/holosoma_retargeting/models/objects/trashcan/trashcan.urdf (robot description, URDF)
Before this commit: robot trashcan.urdf, 1 links, 0 joints
Links:
- link baseLink: mass None -> 0.1
