Commit message: Refactor code structure for improved readability and maintainability

File: src/holosoma_retargeting/holosoma_retargeting/models/r1/r1.urdf (robot description, URDF)
Before this commit: robot r1, 40 links, 39 joints
Links:
- added link left_hand_contact_link, mass 0.001; visual sphere radius=0.015
- added link right_hand_contact_link, mass 0.001; visual sphere radius=0.015
Joints:
- added joint left_hand_contact_joint: type fixed, parent left_wrist_roll_link, child left_hand_contact_link, origin xyz=0.07 0 0 rpy=0 0 0
- added joint right_hand_contact_joint: type fixed, parent right_wrist_roll_link, child right_hand_contact_link, origin xyz=0.07 0 0 rpy=0 0 0

File: src/holosoma_retargeting/holosoma_retargeting/models/r1/r1_26dof.urdf (robot description, URDF)
Before this commit: robot r1_26dof, 48 links, 47 joints
Links:
- added link left_hand_contact_link, mass 0.001; visual sphere radius=0.015
- added link right_hand_contact_link, mass 0.001; visual sphere radius=0.015
Joints:
- added joint left_hand_contact_joint: type fixed, parent left_wrist_roll_link, child left_hand_contact_link, origin xyz=0.07 0 0 rpy=0 0 0
- added joint right_hand_contact_joint: type fixed, parent right_wrist_roll_link, child right_hand_contact_link, origin xyz=0.07 0 0 rpy=0 0 0
