Commit message: Refactor code structure and remove redundant code blocks for improved readability and maintainability

File: src/holosoma_retargeting/holosoma_retargeting/models/r1/r1.urdf (robot description, URDF)
Before this commit: robot r1, 42 links, 41 joints
Joints:
- joint left_hand_contact_joint: origin xyz=0.07 0 0 rpy=0 0 0 -> xyz=0.1 0 0 rpy=0 0 0
- joint right_hand_contact_joint: origin xyz=0.07 0 0 rpy=0 0 0 -> xyz=0.1 0 0 rpy=0 0 0

File: src/holosoma_retargeting/holosoma_retargeting/models/r1/r1_26dof.urdf (robot description, URDF)
Before this commit: robot r1_26dof, 50 links, 49 joints
Joints:
- joint left_hand_contact_joint: origin xyz=0.07 0 0 rpy=0 0 0 -> xyz=0.1 0 0 rpy=0 0 0
- joint right_hand_contact_joint: origin xyz=0.07 0 0 rpy=0 0 0 -> xyz=0.1 0 0 rpy=0 0 0
