Commit message: Add new assets and configurations for whitechair and various RL scenarios
- Created new asset hash file for whitechair.
- Added configuration YAML for whitechair with detailed properties.
- Introduced multiple USD files for whitechair's base, physics, robot, and sensor configurations.
- Added new NPZ files for largebox, plasticbox, smalltable, suitcase, and whitechair scenarios.
- Ensured all new files are properly structured and accessible for simulation tasks.

File: train_r1/objects/resmimicchair/resmimicchair.urdf (robot description, URDF)
Before this commit: robot trashcan.urdf, 1 links, 0 joints
Links:
- link baseLink: geometry collision mesh filename=objects/resmimicchair/resmimicchair.obj scale=1.0 1.0 1.0; visual mesh filename=objects/resmimicchair/resmimicchair.obj scale=1.0 1.0 1.0
