Commit message: Add plasticbox and suitcase object configurations and assets
- Created USD and URDF configurations for the plasticbox object, including robot and sensor definitions.
- Added the plasticbox mesh file and sample points data.
- Introduced suitcase object configurations, including USD files and a YAML configuration for simulation parameters.
- Included physics and sensor definitions for the suitcase object.
- Generated asset hash for suitcase and ensured proper file structure for both objects.

File: train_r1/objects/plasticbox/plasticbox.urdf (robot description, URDF)
Before this commit: robot resmimicchair.urdf, 1 links, 0 joints
Links:
- removed link baseLink
- added link plasticbox_link, mass 0.1; collision mesh filename=objects/plasticbox/plasticbox.obj scale=1.0 1.0 1.0; visual mesh filename=objects/plasticbox/plasticbox.obj scale=1.0 1.0 1.0
